File: KiCad/Practice/Practice.kicad_pcb (KiCad board)
At the start: 4 copper layers, 110 x 70 mm, 37 parts, among them J1 Barrel_Jack_MountingPin, SW1 SW_DIP_x08, SW2 SW_DIP_x01, U1 74AHC273, U2 ICM7555xP

Commit message: Preliminary CAD Design Selected
Parts:
- added G***: LOGO, LOGO, F.Cu at (117.5, 126.5)
- added G***: LOGO, LOGO, B.Cu at (128.2, 85.8)
- moved REF** 21.0 mm to (114.2, 107.8)
- moved G*** 15.1 mm to (114.2, 94.5)
- moved G*** 6.00 mm to (113.0, 94.0)
- moved REF** 4.98 mm to (113.8, 81.5)
- moved G*** 4.04 mm to (200.2, 94.5)
- moved G*** 3.09 mm to (194.0, 118.8)
Other:
- board text added: "Developed by Daniel J. Lomis with Support from AMP Lab Mentor: Professor Jason S. Thweatt"
- board text removed: "Developed by Daniel J. Lomis"
